File: _autosave-matrix.sch (KiCad schematic (older format))
At the start: 124 parts

Commit message: PCB layout
Connections:
- net COL1: no longer D11.1 (K), D15.1 (K), D20.1 (K), D24.1 (K), D28.1 (K), D32.1 (K), D36.1 (K), D41.1 (K), D45.1 (K), D49.1 (K), D5.1 (K), D53.1 (K), D58.1 (K), D62.1 (K)
- new net ROW3: D11.1 (K), D15.1 (K), D20.1 (K), D24.1 (K), D28.1 (K), D32.1 (K), D36.1 (K), D41.1 (K), D45.1 (K), D49.1 (K), D5.1 (K), D53.1 (K), D58.1 (K), D62.1 (K)
Changed lines of the file:
@@
 	8250 5400 8250 4600
 Connection ~ 9350 3000
-Wire Wire Line
-	2400 5050 2750 5050
 Connection ~ 9900 3000
 $Comp
@@
 Wire Wire Line
 	2750 1850 2750 2200
-Wire Wire Line
-	2750 5050 2750 5400
 Wire Wire Line
 	1650 4600 1650 5400
@@
 Wire Wire Line
 	3500 5050 4050 5050
-Connection ~ 3500 5050
-Connection ~ 2400 5050
 Connection ~ 1300 5050
 Wire Wire Line
@@
 Wire Wire Line
 	2400 5850 2950 5850
-Connection ~ 2750 5050
-Wire Wire Line
-	2750 5050 3500 5050
 Wire Wire Line
 	1300 2650 2400 2650
-Wire Wire Line
-	2750 4600 2750 5050
-Connection ~ 2750 4600
 Text Notes 4450 6600 2    50   ~ 0
 Note that MX_ESC1 is placed at the bottom of COL1 instead of recieving its own column.
+Connection ~ 2400 5050
+Connection ~ 3500 5050
+Connection ~ 2750 4600
+Wire Wire Line
+	2400 5050 3500 5050
+Wire Wire Line
+	2750 4600 2750 5400
 $EndSCHEMATC
