File: _autosave-relp65.sch (KiCad schematic (older format))
At the start: 16 parts, among them SW1 SW_Push, U1 ATmega32U4-AU, Y1 16MHz

Commit message: PCB layout
Connections:
- net COL14: now reaches U1.18 (PD0)
- net COL13: now reaches U1.19 (PD1)
- net COL12: now reaches U1.20 (PD2)
- net COL11: now reaches U1.21 (PD3)
- net COL10: now reaches U1.22 (PD5)
- net COL9: now reaches U1.25 (PD4)
- net COL8: now reaches U1.26 (PD6)
- net COL7: now reaches U1.27 (PD7)
- net COL6: now reaches U1.28 (PB4)
- net COL5: now reaches U1.29 (PB5)
- net COL4: now reaches U1.30 (PB6)
- net COL3: now reaches U1.31 (PC6)
- net COL2: now reaches U1.32 (PC7)
- net COL1: now reaches U1.36 (PF7)
- net COL0: now reaches U1.37 (PF6)
- net ROW4: now reaches U1.38 (PF5)
- net ROW3: now reaches U1.39 (PF4)
- net ROW2: now reaches U1.40 (PF1)
- net ROW1: now reaches U1.41 (PF0)
- net ROW0: now reaches U1.8 (PB0)
Changed lines of the file:
@@
 Wire Notes Line
 	3750 5800 5550 5800
+Text GLabel 7400 4800 2    50   Input ~ 0
+ROW4
+Wire Wire Line
+	7400 4800 7150 4800
+Text GLabel 7400 4700 2    50   Input ~ 0
+ROW3
+Text GLabel 7400 4600 2    50   Input ~ 0
+ROW2
+Text GLabel 7400 4500 2    50   Input ~ 0
+ROW1
+Text GLabel 7400 2100 2    50   Input ~ 0
+ROW0
+Wire Wire Line
+	7400 2100 7150 2100
+Wire Wire Line
+	7400 4500 7150 4500
+Wire Wire Line
+	7150 4600 7400 4600
+Wire Wire Line
+	7400 4700 7150 4700
+Text GLabel 7400 4900 2    50   Input ~ 0
+COL0
+Text GLabel 7400 5000 2    50   Input ~ 0
+COL1
+Text GLabel 7450 3100 2    50   Input ~ 0
+COL2
+Text GLabel 7450 3000 2    50   Input ~ 0
+COL3
+Text GLabel 7450 2700 2    50   Input ~ 0
+COL4
+Text GLabel 7450 2600 2    50   Input ~ 0
+COL5
+Text GLabel 7450 2500 2    50   Input ~ 0
+COL6
+Text GLabel 7450 4000 2    50   Input ~ 0
+COL7
+Text GLabel 7450 3900 2    50   Input ~ 0
+COL8
+Text GLabel 7450 3700 2    50   Input ~ 0
+COL9
+Text GLabel 7450 3800 2    50   Input ~ 0
+COL10
+Text GLabel 7450 3600 2    50   Input ~ 0
+COL11
+Text GLabel 7450 3500 2    50   Input ~ 0
+COL12
+Text GLabel 7450 3400 2    50   Input ~ 0
+COL13
+Text GLabel 7450 3300 2    50   Input ~ 0
+COL14
+Wire Wire Line
+	7150 2500 7450 2500
+Wire Wire Line
+	7450 2600 7150 2600
+Wire Wire Line
+	7150 2700 7450 2700
+Wire Wire Line
+	7450 3000 7150 3000
+Wire Wire Line
+	7150 3100 7450 3100
+Wire Wire Line
+	7450 3300 7150 3300
+Wire Wire Line
+	7150 3400 7450 3400
+Wire Wire Line
+	7450 3500 7150 3500
+Wire Wire Line
+	7150 3600 7450 3600
+Wire Wire Line
+	7450 3700 7150 3700
+Wire Wire Line
+	7150 3800 7450 3800
+Wire Wire Line
+	7450 3900 7150 3900
+Wire Wire Line
+	7150 4000 7450 4000
+Wire Wire Line
+	7400 4900 7150 4900
+Wire Wire Line
+	7150 5000 7400 5000
 $EndSCHEMATC
